File: sensor/controller/HackJrGameController-v1.0.sch (EAGLE design)
At the start: 37 parts, among them K1 BUTTON-4P-3110040P1, K2 BUTTON-4P-3110040P1, K3 BUTTON-4P-3110040P1, K4 BUTTON-4P-3110040P1, SW1 SWITCH-2CH-6P-3010010P1, SW2 SWITCH-2CH-6P-3010010P1

Commit message: update schematic, layout and new gerber files for manufacturing
Parts:
- removed D1: LED-RGB-CA-THRUDIFFUSE, SparkFun-LED:LED-RGB-CA-THRUDIFFUSE
- added LED6: RGBLED_CA-5MM, adafruit:RGBLED_CA-5MM
Connections:
- removed net N$21: K1.A0, U$1.*D3
- new net N$40: K1.B0, U$1.*D3
- net N$1: now also LED6.VCC; no longer D1.ANODE, K1.B1, K2.B1, K3.B1, K4.B1, SW1.CH1A, SW2.CH1A
- net N$2: now also SW1.CH1A, SW2.CH1A; no longer U$1.GND@2
- net N$22: now also K2.B0; no longer K2.A0
- net N$23: now also K3.B0; no longer K3.A0
- net N$24: now also K4.B0; no longer K4.A0
- net N$3: now also LED6.RED; no longer D1.RED_CATHODE
- net N$4: now also LED6.BLUE; no longer D1.BLUE_CATHODE
- net N$5: now also LED6.GREEN; no longer D1.GREEN_CATHODE
Other:
- moved on the sheet: K1, K2, K3, K4, SW1, SW2
